Commit message: feat: add 3D RGB camera to agent model
1. Add 3D RGB camera to agent model
2. Updated 3D Camera Library in .gazebo file

File: my_robot/urdf/my_robot.xacro (robot description, xacro)
@@ -121,4 +121,7 @@
    </collision>
  </link>
+  <!--RGB-D Camera-->
+  <link name="camera_link_optical">
+  </link>
  <!--Define Hokuyo Sensor-->
  <link name="hokuyo">
@@ -164,4 +167,9 @@
     <axis xyz="0 1 0" rpy="0 0 0"/>
   </joint>
+ <joint name="camera_optical_joint" type="fixed">
+    <origin xyz="0 0 0" rpy="-1.5707 0 -1.5707"/>
+    <parent link="camera"/>
+    <child link="camera_link_optical"/>
+  </joint>
   <joint type="fixed" name="hokuyo_joint">
     <origin xyz="0.15 0 0.1" rpy="0 0 0"/>
